File: lidar 2/_autosave-lidar 2 round.kicad_pcb (KiCad board)
At the start: 2 copper layers, 60 x 60 mm, 21 parts, among them J1 UART, J2 Motor, J3 JTAG, J4 VIN, J5 USB_C_Receptacle_USB2.0, Q1 BC847, SW1 BOOT, SW2 RESET, U1 AMS1117-5.0, U4 DRV5055A2xDBZxQ1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

Commit message: Made some changes
Parts:
- added LC8805B-1515: ~, led:LC8805B-1515, F.Cu at (130.1, 122.4)
- R3: value 500 Kohm -> 1 Mohm
Connections:
- U5 pad 16: unconnected-(U5-GPIO12/TOUCH12/ADC2_CH1/FSPICLK/FSPIIO6/SUBSPICLK-Pad16) -> SLED
