File: lidar 2/lidar 2 round.kicad_pcb (KiCad board)
At the start: 2 copper layers, 60 x 60 mm, 21 parts, among them J1 UART, J2 Motor, J3 JTAG, J4 VIN, J5 USB_C_Receptacle_USB2.0, Q1 BC847, SW1 BOOT, SW2 RESET, U1 AMS1117-5.0, U4 DRV5055A2xDBZxQ1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

Commit message: More changes
Parts:
- added R4: 1 Mohm, Resistor_SMD:R_0402_1005Metric, F.Cu at (128.3, 90.8)
- added U3: ~, led:LC8805B-1515, F.Cu at (130.3, 131.3)
- R1, R2: footprint Resistor_SMD:R_0805_2012Metric -> Resistor_SMD:R_0402_1005Metric
- R3: value 500 Kohm -> 1 Mohm; footprint Resistor_SMD:R_0805_2012Metric -> Resistor_SMD:R_0402_1005Metric
- moved R2 3.00 mm to (142.2, 97.2), turned to 90 degrees
- moved R3 2.74 mm to (128.3, 92.7)
- moved C1 0.59 mm to (137.8, 97.2)
- moved C3 0.59 mm to (139.8, 97.2)
Connections:
- R3 pad 2: Net-(U5-EN) -> Net-(R3-Pad2)
- SW2 pad 1: Net-(U5-EN) -> Net-(R3-Pad2)
- U5 pad 16: unconnected-(U5-GPIO12/TOUCH12/ADC2_CH1/FSPICLK/FSPIIO6/SUBSPICLK-Pad16) -> SLED
Routing:
- net GND: track 0.00 -> 213.0 mm, vias 0 -> 4
- net +3.3V: track 0.00 -> 97.5 mm, vias 0 -> 6
- net SLED: track 0.00 -> 53.0 mm, vias 0 -> 4
- net TMS: track 0.00 -> 48.4 mm, vias 0 -> 4
- net TDI: track 0.00 -> 45.1 mm, vias 0 -> 4
- net TDO: track 0.00 -> 41.4 mm, vias 0 -> 4
- net D-: track 0.00 -> 41.2 mm, vias 0 -> 6
- net D+: track 0.00 -> 40.8 mm, vias 0 -> 7
- net Hall_Effect_Sensor: track 0.00 -> 38.6 mm, vias 0 -> 6
- net TCK: track 0.00 -> 37.7 mm, vias 0 -> 4
- net +5V: track 0.00 -> 35.9 mm, vias 0 -> 1
- net TX: track 0.00 -> 32.5 mm
- net RX: track 0.00 -> 31.6 mm
- net Net-(U5-EN): track 0.00 -> 29.1 mm, vias 0 -> 2
- net SCL: track 0.00 -> 26.4 mm, vias 0 -> 2
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
Commit message: Finsished mk2
Parts:
- added H1: MountingHole_Pad, MountingHole:MountingHole_2.2mm_M2, F.Cu at (157.5, 119.9)
- added H2: MountingHole_Pad, MountingHole:MountingHole_2.2mm_M2, F.Cu at (157.5, 78.7)
- added H3: MountingHole_Pad, MountingHole:MountingHole_2.2mm_M2, F.Cu at (120.9, 78.7)
- added H5: MountingHole_Pad, MountingHole:MountingHole_2.2mm_M2, F.Cu at (120.9, 119.9)
- USB C: renamed from J5
- renumbered U6 to +3v3, U1 to +5V
Routing:
- net Net-(U5-GPIO0/BOOT): track 0.00 -> 22.5 mm, vias 0 -> 2
- net SLED: track 53.0 -> 50.7 mm
- added copper zone on F.Cu, net GND
Other:
- board text added: "+ -"
- board text added: "3v3 RX TX GND"
- board text added: "BOOT"
- board text added: "GOOD LIDAR"
- board text added: "HALL EFFECT SENSOR"
- board text added: "JTAG"
- board text added: "MOTOR"
- board text added: "RESET"
- board text added: "STATUS"
- board text added: "TCK TDO TDI TMS"
- board text added: "Time of Flight"
- board text added: "UART"
