File: lidar 2/lidar 2 round.kicad_sch (KiCad schematic)
At the start: 20 parts, among them J1 USB_C_Receptacle_USB2.0, J2 Motor, J3 UART, J4 JTAG, J5 VIN, Q2 BC847, SW1 BOOT, SW2 RESET, U1 LM1117DT-3.3, U2 LM1117S-5.0, U3 ESP32-S3-MINI-1, U6 DRV5055A2xDBZxQ1

Commit message: Made some changes
Parts:
- removed SW2: RESET, Button_Switch_SMD:SW_Push_1P1T_NO_6x6mm_H9.5mm, symbol Switch:SW_Push_Open
- removed U1: LM1117DT-3.3, Package_TO_SOT_SMD:TO-252-3_TabPin2, symbol Regulator_Linear:LM1117DT-3.3
- removed U2: LM1117S-5.0, Package_TO_SOT_SMD:TO-263-3_TabPin2, symbol Regulator_Linear:LM1117S-5.0
- added R? (x2): 1 Mohm, Resistor_SMD:R_0805_2012Metric, symbol Device:R_Small
- added SW?: RESET, Button_Switch_SMD:SW_Push_SPST_NO_Alps_SKRK, symbol Switch:SW_Push
- added U1: AMS1117-5.0, Package_TO_SOT_SMD:SOT-223-3_TabPin2, symbol Regulator_Linear:AMS1117-5.0
- added U3: ~, led:LC8805B-1515, symbol LC8805:LC8805B-1515
- added U6: AMS1117-3.3, Package_TO_SOT_SMD:SOT-223-3_TabPin2, symbol Regulator_Linear:AMS1117-3.3
- J?: renamed from J1; footprint Connector_USB:USB_C_Receptacle_GCT_USB4110 -> Connector_USB:USB_C_Receptacle_Amphenol_12401610E4-2A
- SW?: renamed from SW1; footprint Button_Switch_SMD:SW_Push_1P1T_NO_6x6mm_H9.5mm -> Button_Switch_SMD:SW_Push_SPST_NO_Alps_SKRK
- renumbered D1 to D?, J3 to J1, J4 to J3, J5 to J4, Q2 to Q1, R2 to R?, R1 to R?, U4 to U2, U6 to U4, U3 to U?
Connections:
- net +3.3V: now also R?.1, U3. (VDD), U6.2 (VO)
- net +5V: now also U1.2 (VO)
- net GND: now also SW?.2, U1.1 (GND), U3. (VDD), U6.1 (GND)
- net VIN: now also U1.3 (VI), U6.3 (VI)
- net at U?.45 (EN): now also R?.2
- net SLED: now reaches U?.16 (GPIO12/TOUCH12/ADC2_CH1/FSPICLK/FSPIIO6/SUBSPICLK)
- net SLED: now also U3. (VDD)
- new net: R?.1, R?.2, SW?.1
Other:
- note added: "Figure out resistance"
- moved on the sheet: J4

Commit message: More changes
Parts:
- R? (x4): footprint Resistor_SMD:R_0805_2012Metric -> Resistor_SMD:R_0402_1005Metric
Connections:
- net +3.3V: now also U3.2 (VDD); no longer U3. (VDD)
- net GND: now also U3.4 (GND); no longer U3. (VDD)
- net SLED: now also U3.1 (DIN); no longer U3. (VDD)
Changed lines of the file:
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@@
+    )
+  )
+  (global_label "SLED" (shape input) (at 93.98 140.97 180) (fields_autoplaced)
+    (effects (font (size 1.27 1.27)) (justify right))
+    (property "Intersheetrefs" "${INTERSHEET_REFS}" (at 86.3382 140.97 0)
+      (effects (font (size 1.27 1.27)) (justify right) hide)
     )
   )
@@
     )
   )
-  (global_label "SLED" (shape input) (at 93.98 140.97 180) (fields_autoplaced)
-    (effects (font (size 1.27 1.27)) (justify right))
-    (property "Intersheetrefs" "${INTERSHEET_REFS}" (at 86.3382 140.97 0)
-      (effects (font (size 1.27 1.27)) (justify right) hide)
-    )
-  )
   (global_label "D-" (shape input) (at 128.27 62.23 0) (fields_autoplaced)
     (effects (font (size 1.27 1.27)) (justify left))
@@
       (effects (font (size 1.27 1.27)))
     )
-    (property "Footprint" "Resistor_SMD:R_0805_2012Metric" (at 262.89 124.46 0)
+    (property "Footprint" "Resistor_SMD:R_0402_1005Metric" (at 262.89 124.46 0)
       (effects (font (size 1.27 1.27)) hide)
     )
@@
         (path "/dd34a7c1-47d4-480b-86be-f1ea16fc4df3"
           (reference "R3") (unit 1)
-        )
-      )
-    )
-  )
-  (symbol (lib_id "power:+5V") (at 59.69 111.76 270) (unit 1)
-    (in_bom yes) (on_board yes) (dnp no) (fields_autoplaced)
-    (property "Reference" "#PWR?" (at 55.88 111.76 0)
-      (effects (font (size 1.27 1.27)) hide)
-    )
-    (property "Value" "+5V" (at 63.5 111.76 90)
-      (effects (font (size 1.27 1.27)) (justify left))
-    )
-    (property "Footprint" "" (at 59.69 111.76 0)
-      (effects (font (size 1.27 1.27)) hide)
-    )
-    (property "Datasheet" "" (at 59.69 111.76 0)
-      (effects (font (size 1.27 1.27)) hide)
-    )
-    (pin "1")
-    (instances
-      (project "lidar"
-        (path "/2624fe18-dd3c-43e6-b135-e885653f3dbb"
-          (reference "#PWR?") (unit 1)
-        )
-      )
-      (project "lidar 2 round"
-        (path "/dd34a7c1-47d4-480b-86be-f1ea16fc4df3"
-          (reference "#PWR010") (unit 1)
         )
       )
@@
         (path "/dd34a7c1-47d4-480b-86be-f1ea16fc4df3"
           (reference "#PWR028") (unit 1)
-        )
-      )
-    )
-  )
-  (symbol (lib_id "LC8805:LC8805B-1515") (at 101.6 137.16 0) (unit 1)
-    (in_bom yes) (on_board yes) (dnp no) (fields_autoplaced)
-    (property "Reference" "U3" (at 101.6 133.35 0)
-      (effects (font (size 1.27 1.27)))
-    )
-    (property "Value" "~" (at 101.6 137.16 0)
-      (effects (font (size 1.27 1.27)))
-    )
-    (property "Footprint" "led:LC8805B-1515" (at 101.6 134.62 0)
-      (effects (font (size 1.27 1.27)) hide)
-    )
-    (property "Datasheet" "" (at 101.6 137.16 0)
-      (effects (font (size 1.27 1.27)) hide)
-    )
-    (pin "")
-    (pin "")
-    (pin "")
-    (pin "")
-    (instances
-      (project "lidar 2 round"
-        (path "/dd34a7c1-47d4-480b-86be-f1ea16fc4df3"
-          (reference "U3") (unit 1)
         )
       )
@@
     )
   )
+  (symbol (lib_id "LC8805:LC8805B-1515") (at 101.6 137.16 0) (unit 1)
+    (in_bom yes) (on_board yes) (dnp no) (fields_autoplaced)
+    (property "Reference" "U3" (at 101.6 133.35 0)
+      (effects (font (size 1.27 1.27)))
+    )
+    (property "Value" "~" (at 101.6 137.16 0)
+      (effects (font (size 1.27 1.27)))
+    )
+    (property "Footprint" "led:LC8805B-1515" (at 101.6 134.62 0)
+      (effects (font (size 1.27 1.27)) hide)
+    )
+    (property "Datasheet" "" (at 101.6 137.16 0)
+      (effects (font (size 1.27 1.27)) hide)
+    )
+    (pin "3")
+    (pin "4")
+    (pin "2")
+    (pin "1")
+    (instances
+      (project "lidar 2 round"
+        (path "/dd34a7c1-47d4-480b-86be-f1ea16fc4df3"
+          (reference "U3") (unit 1)
+        )
+      )
+    )
+  )
   (symbol (lib_id "power:+3.3V") (at 48.26 46.99 270) (unit 1)
     (in_bom yes) (on_board yes) (dnp no) (fields_autoplaced)
@@
       (effects (font (size 1.27 1.27)))
     )
-    (property "Footprint" "Resistor_SMD:R_0805_2012Metric" (at 260.35 121.92 0)
+    (property "Footprint" "Resistor_SMD:R_0402_1005Metric" (at 260.35 121.92 0)
       (effects (font (size 1.27 1.27)) hide)
     )
@@
       (effects (font (size 1.27 1.27)))
     )
-    (property "Footprint" "Resistor_SMD:R_0805_2012Metric" (at 34.29 120.65 0)
+    (property "Footprint" "Resistor_SMD:R_0402_1005Metric" (at 34.29 120.65 0)
       (effects (font (size 1.27 1.27)) hide)
     )
@@
       (effects (font (size 1.27 1.27)))
     )
-    (property "Footprint" "Resistor_SMD:R_0805_2012Metric" (at 83.82 81.28 0)
+    (property "Footprint" "Resistor_SMD:R_0402_1005Metric" (at 83.82 81.28 0)
       (effects (font (size 1.27 1.27)) hide)
     )
@@
         )
       )
+    )
+  )
+  (symbol (lib_id "power:+5V") (at 59.69 111.76 270) (unit 1)
+    (in_bom yes) (on_board yes) (dnp no) (fields_autoplaced)
+    (property "Reference" "#PWR?" (at 55.88 111.76 0)
+      (effects (font (size 1.27 1.27)) hide)
+    )
+    (property "Value" "+5V" (at 63.5 111.76 90)
+      (effects (font (size 1.27 1.27)) (justify left))
+    )
+    (property "Footprint" "" (at 59.69 111.76 0)
+      (effects (font (size 1.27 1.27)) hide)
+    )
+    (property "Datasheet" "" (at 59.69 111.76 0)
+      (effects (font (size 1.27 1.27)) hide)
+    )
+    (pin "1")
+    (instances
+      (project "lidar"
+        (path "/2624fe18-dd3c-43e6-b135-e885653f3dbb"
+          (reference "#PWR?") (unit 1)
+        )
+      )
+      (project "lidar 2 round"
+        (path "/dd34a7c1-47d4-480b-86be-f1ea16fc4df3"
+          (reference "#PWR010") (unit 1)
+        )
+      )

Commit message: Finsished mk2
Parts:
- added H1, H2, H3, H5: MountingHole_Pad, MountingHole:MountingHole_2.2mm_M2, symbol Mechanical:MountingHole_Pad
Changed lines of the file:
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@@
+    )
+  )
+  (symbol (lib_id "Mechanical:MountingHole_Pad") (at 24.13 173.99 270) (unit 1)
+    (in_bom yes) (on_board yes) (dnp no) (fields_autoplaced)
+    (property "Reference" "H3" (at 27.94 172.72 90)
+      (effects (font (size 1.27 1.27)) (justify left))
+    )
+    (property "Value" "MountingHole_Pad" (at 27.94 175.26 90)
+      (effects (font (size 1.27 1.27)) (justify left))
+    )
+    (property "Footprint" "MountingHole:MountingHole_2.2mm_M2" (at 24.13 173.99 0)
+      (effects (font (size 1.27 1.27)) hide)
+    )
+    (property "Datasheet" "~" (at 24.13 173.99 0)
+      (effects (font (size 1.27 1.27)) hide)
+    )
+    (pin "1")
+    (instances
+      (project "lidar 2 round"
+        (path "/dd34a7c1-47d4-480b-86be-f1ea16fc4df3"
+          (reference "H3") (unit 1)
+        )
+      )
+    )
+  )
+  (symbol (lib_id "Mechanical:MountingHole_Pad") (at 24.13 163.83 270) (unit 1)
+    (in_bom yes) (on_board yes) (dnp no) (fields_autoplaced)
+    (property "Reference" "H1" (at 27.94 162.56 90)
+      (effects (font (size 1.27 1.27)) (justify left))
+    )
+    (property "Value" "MountingHole_Pad" (at 27.94 165.1 90)
+      (effects (font (size 1.27 1.27)) (justify left))
+    )
+    (property "Footprint" "MountingHole:MountingHole_2.2mm_M2" (at 24.13 163.83 0)
+      (effects (font (size 1.27 1.27)) hide)
+    )
+    (property "Datasheet" "~" (at 24.13 163.83 0)
+      (effects (font (size 1.27 1.27)) hide)
+    )
+    (pin "1")
+    (instances
+      (project "lidar 2 round"
+        (path "/dd34a7c1-47d4-480b-86be-f1ea16fc4df3"
+          (reference "H1") (unit 1)
+        )
+      )
     )
   )
@@
         (path "/dd34a7c1-47d4-480b-86be-f1ea16fc4df3"
           (reference "#PWR028") (unit 1)
+        )
+      )
+    )
+  )
+  (symbol (lib_id "Mechanical:MountingHole_Pad") (at 24.13 158.75 270) (unit 1)
+    (in_bom yes) (on_board yes) (dnp no) (fields_autoplaced)
+    (property "Reference" "H5" (at 27.94 157.48 90)
+      (effects (font (size 1.27 1.27)) (justify left))
+    )
+    (property "Value" "MountingHole_Pad" (at 27.94 160.02 90)
+      (effects (font (size 1.27 1.27)) (justify left))
+    )
+    (property "Footprint" "MountingHole:MountingHole_2.2mm_M2" (at 24.13 158.75 0)
+      (effects (font (size 1.27 1.27)) hide)
+    )
+    (property "Datasheet" "~" (at 24.13 158.75 0)
+      (effects (font (size 1.27 1.27)) hide)
+    )
+    (pin "1")
+    (instances
+      (project "lidar 2 round"
+        (path "/dd34a7c1-47d4-480b-86be-f1ea16fc4df3"
+          (reference "H5") (unit 1)
         )
       )
@@
         )
       )
+    )
+  )
+  (symbol (lib_id "Mechanical:MountingHole_Pad") (at 24.13 168.91 270) (unit 1)
+    (in_bom yes) (on_board yes) (dnp no) (fields_autoplaced)
+    (property "Reference" "H2" (at 27.94 167.64 90)
+      (effects (font (size 1.27 1.27)) (justify left))
+    )
+    (property "Value" "MountingHole_Pad" (at 27.94 170.18 90)
+      (effects (font (size 1.27 1.27)) (justify left))
+    )
+    (property "Footprint" "MountingHole:MountingHole_2.2mm_M2" (at 24.13 168.91 0)
+      (effects (font (size 1.27 1.27)) hide)
+    )
+    (property "Datasheet" "~" (at 24.13 168.91 0)
+      (effects (font (size 1.27 1.27)) hide)
+    )
+    (pin "1")
+    (instances
+      (project "lidar 2 round"
+        (path "/dd34a7c1-47d4-480b-86be-f1ea16fc4df3"
+          (reference "H2") (unit 1)
+        )
+      )
